Commit message: added multiple sensors and gazebo world to simulate the bot on

File: description/Arm.xacro (robot description, xacro)
@@ -4,4 +4,9 @@
 <xacro:include filename="$(find spatial_manipulator)/description/Arm.trans" />
 <xacro:include filename="$(find spatial_manipulator)/description/Arm.gazebo" />
+<joint name="arm_joint" type="fixed">
+    <parent link="chassis_link"/>
+    <child link="arm_base_link"/>
+    <origin xyz="0.15 0.0 0.2" rpy="0.0 0.0 ${pi}"/>
+</joint>
 <link name="arm_base_link">
   <inertial>

File: description/robot.urdf.xacro (robot description, xacro)
@@ -3,4 +3,7 @@
     <xacro:include filename="robot_core.xacro"/>
     <xacro:include filename="gazebo_control.xacro"/>
-    <!-- <xacro:include filename="lidar.xacro/> -->
+    <xacro:include filename="lidar.xacro"/>
+    <!-- <xacro:include filename="camera.xacro"/> -->
+    <xacro:include filename="depth_camera.xacro"/>
+    <xacro:include filename="imu.xacro"/>
 </robot>

File: description/robot_core.xacro (robot description, xacro)
@@ -3,5 +3,5 @@
     <xacro:include filename="material.xacro"/>
     <xacro:include filename="inertial_macros.xacro" />
-    <xacro:include filename="Arm.xacro" />
+    <!-- <xacro:include filename="Arm.xacro" /> -->
     <link name="base_link">
     </link>
@@ -33,10 +33,36 @@
         <material>Gazebo/Blue</material>
     </gazebo>
+    <!--          LEFT WHEEL           -->
+    <joint name="left_wheel_joint" type="continuous">
+        <origin xyz="0.0 0.28 0.0" rpy="-${pi/2} 0.0 0.0" />
+        <parent link="base_link" />
+        <child link="left_wheel_link" />
+        <axis xyz="0.0 0.0 1" />
+    </joint>
+    <link name="left_wheel_link">
+        <visual>
+            <geometry>
+                <cylinder radius="0.08" length="0.05" />
+            </geometry>
+            <material name="orange" />
+        </visual>
+        <collision>
+            <geometry>
+                <cylinder radius="0.08" length="0.05" />
+            </geometry>
+        </collision>
+        <xacro:inertial_cylinder mass="0.5" length="0.05" radius="0.08">
+            <origin xyz="0 0 0" rpy="0 0 0" />
+        </xacro:inertial_cylinder>
+    </link>
+    <gazebo reference="left_wheel_link">
+        <material>Gazebo/Orange</material>
+    </gazebo>
     <!--          RIGHT WHEEL           -->
     <joint name="right_wheel_joint" type="continuous">
-        <origin xyz="0.0 0.28 0.0" rpy="-${pi/2} 0.0 0.0" />
         <parent link="base_link" />
         <child link="right_wheel_link" />
-        <axis xyz="0.0 0.0 1" />
+        <origin xyz="0.0 -0.28 0.0" rpy="${pi/2} 0.0 0.0" />
+        <axis xyz="0.0 0.0 -1" />
     </joint>
     <link name="right_wheel_link">
@@ -57,30 +83,4 @@
     </link>
     <gazebo reference="right_wheel_link">
-        <material>Gazebo/Green</material>
-    </gazebo>
-    <!--          LEFT WHEEL           -->
-    <joint name="left_wheel_joint" type="continuous">
-        <parent link="base_link" />
-        <child link="left_wheel_link" />
-        <origin xyz="0.0 -0.28 0.0" rpy="${pi/2} 0.0 0.0" />
-        <axis xyz="0.0 0.0 -1" />
-    </joint>
-    <link name="left_wheel_link">
-        <visual>
-            <geometry>
-                <cylinder radius="0.08" length="0.05" />
-            </geometry>
-            <material name="green" />
-        </visual>
-        <collision>
-            <geometry>
-                <cylinder radius="0.08" length="0.05" />
-            </geometry>
-        </collision>
-        <xacro:inertial_cylinder mass="0.5" length="0.05" radius="0.08">
-            <origin xyz="0 0 0" rpy="0 0 0" />
-        </xacro:inertial_cylinder>
-    </link>
-    <gazebo reference="left_wheel_link">
         <material>Gazebo/Green</material>
     </gazebo>
@@ -136,9 +136,3 @@
         <mu2 value="0.01" />
     </gazebo>
-    <!--                               Robotic ARM                                      -->
-    <joint name="arm_joint" type="fixed">
-        <parent link="chassis_link"/>
-        <child link="arm_base_link"/>
-        <origin xyz="0.25 0.0 0.2" rpy="0.0 0.0 ${pi}"/>
-    </joint>
 </robot>
