Commit message: added ros2 control for differential drive bot and improved readme

File: description/imu.xacro (robot description, xacro)
@@ -25,5 +25,5 @@
             <plugin name="imu_plugin" filename="libgazebo_ros_imu_sensor.so">
                 <frame_name>imu_link</frame_name>
-                <initialOrientationAsReference>false</initialOrientationAsReference>
+                <initial_orientation_as_reference>false</initial_orientation_as_reference>
             </plugin>
         </sensor>

File: description/robot.urdf.xacro (robot description, xacro)
@@ -1,9 +1,15 @@
 <?xml version="1.0"?>
 <robot xmlns:xacro="http://www.ros.org/wiki/xacro" name="spatial_manipulator">
-    <xacro:include filename="robot_core.xacro"/>
-    <xacro:include filename="gazebo_control.xacro"/>
-    <xacro:include filename="lidar.xacro"/>
+    <xacro:arg name="use_ros2_control" default="true" />
+    <xacro:include filename="robot_core.xacro" />
+    <xacro:if value="$(arg use_ros2_control)">
+        <xacro:include filename="ros2_control.xacro" />
+    </xacro:if>
+    <xacro:unless value="$(arg use_ros2_control)">
+        <xacro:include filename="gazebo_control.xacro"/>
+    </xacro:unless>
+    <xacro:include filename="lidar.xacro" />
     <!-- <xacro:include filename="camera.xacro"/> -->
-    <xacro:include filename="depth_camera.xacro"/>
-    <xacro:include filename="imu.xacro"/>
+    <xacro:include filename="depth_camera.xacro" />
+    <xacro:include filename="imu.xacro" />
 </robot>

File: description/robot_core.xacro (robot description, xacro)
@@ -1,5 +1,5 @@
 <?xml version="1.0"?>
 <robot xmlns:xacro="http://www.ros.org/wiki/xacro">
-    <xacro:include filename="material.xacro"/>
+    <xacro:include filename="material.xacro" />
     <xacro:include filename="inertial_macros.xacro" />
     <!-- <xacro:include filename="Arm.xacro" /> -->
@@ -49,5 +49,5 @@
         <collision>
             <geometry>
-                <cylinder radius="0.08" length="0.05" />
+                <sphere radius="0.08" />
             </geometry>
         </collision>
@@ -75,5 +75,5 @@
         <collision>
             <geometry>
-                <cylinder radius="0.08" length="0.05" />
+                <sphere radius="0.08" />
             </geometry>
         </collision>
