Commit message: Addition of SLAM using slam_toolbox and nav2_amcl and navigation using nav2

File: description/robot_core.xacro (robot description, xacro)
@@ -5,4 +5,11 @@
     <!-- <xacro:include filename="Arm.xacro" /> -->
     <link name="base_link">
+    </link>
+    <joint name="base_footprint_joint" type="fixed">
+        <origin xyz="0.0 0.0 0.0" rpy="0.0 0.0 0.0"/>
+        <parent link="base_link"/>
+        <child link="base_footprint"/>
+    </joint>
+    <link name="base_footprint">
     </link>
     <!--          CHASSIS           -->
