Commit message: Integration of Moveit with the robot.

File: description/arm.xacro (robot description, xacro)
@@ -2,6 +2,6 @@
 <robot xmlns:xacro="http://www.ros.org/wiki/xacro">
 <!-- <xacro:include filename="material.xacro"/> -->
-<xacro:include filename="$(find spatial_manipulator)/description/Arm.trans" />
-<xacro:include filename="$(find spatial_manipulator)/description/Arm.gazebo" />
+<xacro:include filename="$(find spatial_manipulator)/description/arm.trans" />
+<xacro:include filename="$(find spatial_manipulator)/description/arm.gazebo" />
 <joint name="arm_joint" type="fixed">
     <parent link="chassis_link"/>
@@ -12,5 +12,5 @@
   <inertial>
     <origin xyz="-3.0728641490355835e-17 0.0 0.026990189047542933" rpy="0 0 0"/>
-    <mass value="1.2786172512351936"/>
+    <mass value="0.639308626"/>
     <inertia ixx="0.095069" iyy="0.095069" izz="0.183045" ixy="-0.0" iyz="0.0" ixz="-0.0"/>
   </inertial>
@@ -32,5 +32,5 @@
   <inertial>
     <origin xyz="0.0046856299908202255 0.0 0.14324873354490847" rpy="0 0 0"/>
-    <mass value="0.6118703329147364"/>
+    <mass value="0.305935166"/>
     <inertia ixx="0.044972" iyy="0.045488" izz="0.008164" ixy="0.0" iyz="0.0" ixz="-0.003204"/>
   </inertial>
@@ -52,5 +52,5 @@
   <inertial>
     <origin xyz="0.05770282693838659 -7.870356960513597e-18 0.25623073545187974" rpy="0 0 0"/>
-    <mass value="1.2480428560519359"/>
+    <mass value="0.624021428"/>
     <inertia ixx="0.364873" iyy="0.365457" izz="0.016185" ixy="0.0" iyz="0.0" ixz="-0.00749"/>
   </inertial>
@@ -72,5 +72,5 @@
   <inertial>
     <origin xyz="-0.01372020432066895 4.67375539046592e-09 0.04627975967090037" rpy="0 0 0"/>
-    <mass value="0.2089611133364475"/>
+    <mass value="0.104480557"/>
     <inertia ixx="0.002869" iyy="0.003125" izz="0.002869" ixy="0.0" iyz="-0.0" ixz="0.000537"/>
   </inertial>
@@ -92,5 +92,5 @@
   <inertial>
     <origin xyz="-0.057166086937035156 -0.002833849284401173 0.20000001558393898" rpy="0 0 0"/>
-    <mass value="1.0116831617121436"/>
+    <mass value="0.505841581"/>
     <inertia ixx="0.193829" iyy="0.193829" izz="0.013784" ixy="-8.1e-05" iyz="0.005878" ixz="0.005878"/>
   </inertial>
@@ -112,5 +112,5 @@
   <inertial>
     <origin xyz="0.005039788511788848 -0.05078102194423177 1.5583935253360437e-08" rpy="0 0 0"/>
-    <mass value="0.24108268648902764"/>
+    <mass value="0.120541343"/>
     <inertia ixx="0.002894" iyy="0.006872" izz="0.008175" ixy="0.00078" iyz="0.0" ixz="2e-05"/>
   </inertial>
@@ -132,5 +132,5 @@
   <inertial>
     <origin xyz="0.010000023866328533 -0.024999959122409626 -0.024999984416064658" rpy="0 0 0"/>
-    <mass value="0.013499999999999998"/>
+    <mass value="0.00675"/>
     <inertia ixx="5.6e-05" iyy="3.3e-05" izz="3.3e-05" ixy="-0.0" iyz="0.0" ixz="0.0"/>
   </inertial>
@@ -154,5 +154,5 @@
   <child link="first_link_1"/>
   <axis xyz="0.0 0.0 1.0"/>
-  <limit upper="3.141593" lower="-3.141593" effort="100" velocity="100"/>
+  <limit upper="3.141593" lower="-3.141593" effort="100" velocity="100.0"/>
 </joint>
 <joint name="second_joint" type="revolute">
@@ -161,5 +161,5 @@
   <child link="second_link_1"/>
   <axis xyz="1.0 0.0 0.0"/>
-  <limit upper="2.094395" lower="0.0" effort="100" velocity="100"/>
+  <limit upper="2.094395" lower="0.0" effort="100" velocity="100.0"/>
 </joint>
 <joint name="third_joint" type="revolute">

File: description/robot.urdf.xacro (robot description, xacro)
@@ -9,4 +9,5 @@
         <xacro:include filename="gazebo_control.xacro"/>
     </xacro:unless>
+    <xacro:include filename="arm.xacro" />
     <xacro:include filename="lidar.xacro" />
     <!-- <xacro:include filename="camera.xacro"/> -->

File: description/robot_core.xacro (robot description, xacro)
@@ -3,5 +3,4 @@
     <xacro:include filename="material.xacro" />
     <xacro:include filename="inertial_macros.xacro" />
-    <!-- <xacro:include filename="Arm.xacro" /> -->
     <link name="base_link">
     </link>
@@ -59,5 +58,5 @@
             </geometry>
         </collision>
-        <xacro:inertial_cylinder mass="0.5" length="0.05" radius="0.08">
+        <xacro:inertial_cylinder mass="0.9" length="0.05" radius="0.08">
             <origin xyz="0 0 0" rpy="0 0 0" />
         </xacro:inertial_cylinder>
@@ -85,5 +84,5 @@
             </geometry>
         </collision>
-        <xacro:inertial_cylinder mass="0.5" length="0.05" radius="0.08">
+        <xacro:inertial_cylinder mass="0.9" length="0.05" radius="0.08">
             <origin xyz="0 0 0" rpy="0 0 0" />
         </xacro:inertial_cylinder>
@@ -110,5 +109,5 @@
             </geometry>
         </collision>
-        <xacro:inertial_cylinder mass="0.2" length="0.05" radius="0.04">
+        <xacro:inertial_cylinder mass="0.5" length="0.05" radius="0.04">
             <origin xyz="0 0 0" rpy="0 0 0" />
         </xacro:inertial_cylinder>
@@ -134,5 +133,5 @@
             </geometry>
         </collision>
-        <xacro:inertial_sphere mass="0.6" radius="0.03">
+        <xacro:inertial_sphere mass="0.8" radius="0.03">
             <origin xyz="0 0 0" rpy="0 0 0" />
         </xacro:inertial_sphere>

File: description/ros2_control.xacro (robot description, xacro)
@@ -5,4 +5,5 @@
             <plugin>gazebo_ros2_control/GazeboSystem</plugin>
         </hardware>
+        <!-- DIFF_DRIVE_JOINTS -->
         <joint name="left_wheel_joint">
             <command_interface name="velocity">
@@ -25,4 +26,71 @@
             </state_interface>
         </joint>
+        <!-- ARM_JOINT -->
+        <joint name="first_joint">
+            <command_interface name="position">
+                <param name="min">-3.141593</param>
+                <param name="max">3.141593</param>
+            </command_interface>
+            <state_interface name="position">
+                <param name="initial_value">0.0</param>
+            </state_interface>
+            <state_interface name="velocity"></state_interface>
+            <state_interface name="effort"></state_interface>
+        </joint>
+        <joint name="second_joint">
+            <command_interface name="position">
+                <param name="min">0.0</param>
+                <param name="max">2.094395</param>
+            </command_interface>
+            <state_interface name="position">
+                <param name="initial_value">0.0</param>
+            </state_interface>
+            <state_interface name="velocity"></state_interface>
+            <state_interface name="effort"></state_interface>
+        </joint>
+        <joint name="third_joint">
+            <command_interface name="position">
+                <param name="min">-3.141593</param>
+                <param name="max">3.141593</param>
+            </command_interface>
+            <state_interface name="position">
+                <param name="initial_value">0.0</param>
+            </state_interface>
+            <state_interface name="velocity"></state_interface>
+            <state_interface name="effort"></state_interface>
+        </joint>
+        <joint name="fourth_joint">
+            <command_interface name="position">
+                <param name="min">-2.094395</param>
+                <param name="max">2.094395</param>
+            </command_interface>
+            <state_interface name="position">
+                <param name="initial_value">0.0</param>
+            </state_interface>
+            <state_interface name="velocity"></state_interface>
+            <state_interface name="effort"></state_interface>
+        </joint>
+        <joint name="fifth_joint">
+            <command_interface name="position">
+                <param name="min">-3.141593</param>
+                <param name="max">3.141593</param>
+            </command_interface>
+            <state_interface name="position">
+                <param name="initial_value">0.0</param>
+            </state_interface>
+            <state_interface name="velocity"></state_interface>
+            <state_interface name="effort"></state_interface>
+        </joint>
+        <joint name="gripper_joint">
+            <command_interface name="position">
+                <param name="min">-0.15</param>
+                <param name="max">0.0</param>
+            </command_interface>
+            <state_interface name="position">
+                <param name="initial_value">0.0</param>
+            </state_interface>
+            <state_interface name="velocity"></state_interface>
+            <state_interface name="effort"></state_interface>
+        </joint>
     </ros2_control>
     <gazebo>
